Commit message: Updating contact sensor

File: p_g11_description/urdf/p_g11.gazebo.xacro (robot description, xacro)
@@ -169,7 +169,17 @@
     </sensor>
   </gazebo>
-<!--  Added by me-->
-<!--  <gazebo reference="appendix_box">-->
-<!--    <material>Gazebo/Blue</material>-->
-<!--  </gazebo>-->
+<!--  Contact sensor - added by me -->
+<gazebo reference="base_link">
+    <sensor name="base_link" type="contact">
+      <update_rate>1000.0</update_rate>
+      <always_on>true</always_on>
+      <contact>
+        <collision> "base_footprint_fixed_joint_lump__base_link_collision" </collision>
+      </contact>
+      <plugin name="base_link_contact_sensor_plugin" filename="libgazebo_ros_bumper.so">
+        <bumperTopicName>contact</bumperTopicName>
+        <frameName>world</frameName>
+      </plugin>
+    </sensor>
+  </gazebo>
 </robot>

Commit message: Updating contact sensor

File: p_g11_description/urdf/p_g11.gazebo.xacro (robot description, xacro)
@@ -175,5 +175,5 @@
       <always_on>true</always_on>
       <contact>
-        <collision> "base_footprint_fixed_joint_lump__base_link_collision" </collision>
+        <collision>base_footprint_fixed_joint_lump__base_link_collision</collision>
       </contact>
       <plugin name="base_link_contact_sensor_plugin" filename="libgazebo_ros_bumper.so">
